File: kicad/bandfilter.kicad_pcb (KiCad board)
At the start: 2 copper layers, 152 x 93.7 mm, 106 parts, among them J1 Antenna, J2 Rx, J3 Tx, J4 Conn_01x07, J5 Conn_01x07, J6 Antenna, J7 Rx, J8 Tx, T1 40/13T T50-2 (8uH), T2 30/8T T50-2 (4.5uH)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

Commit message: I2C version update
Parts:
- added C58: 10u, Capacitor_SMD:C_1206_3216Metric_Pad1.42x1.75mm_HandSolder, F.Cu at (196.7, 70.2)
- added C59: 10u, Capacitor_SMD:C_1206_3216Metric_Pad1.42x1.75mm_HandSolder, F.Cu at (196.0, 25.1)
- added C60: 100n, Capacitor_SMD:C_1206_3216Metric_Pad1.42x1.75mm_HandSolder, F.Cu at (131.1, 109.7)
- added C71: 100n, Capacitor_SMD:C_1206_3216Metric_Pad1.42x1.75mm_HandSolder, F.Cu at (147.3, 108.6)
- added U12: AS169-73LF, Package_TO_SOT_SMD:SOT-23-6_Handsoldering, F.Cu at (138.7, 110.7)
- C11: footprint Capacitor_THT:C_Disc_D9.0mm_W2.5mm_P5.00mm -> Capacitor_THT:C_Disc_D9.0mm_W5.0mm_P5.00mm
- C6: footprint Capacitor_THT:C_Disc_D9.0mm_W2.5mm_P5.00mm -> Capacitor_SMD:C_0805_2012Metric_Pad1.15x1.40mm_HandSolder
- U10, U11: value 74HC595 -> PCF8574A; footprint Package_DIP:DIP-16_W7.62mm_Socket -> Package_SO:SOP-16_7.5x10.4mm_P1.27mm
- moved U11 23.2 mm to (189.4, 77.3)
- moved C66 15.6 mm to (196.7, 67.1)
- moved C48 9.59 mm to (198.6, 25.1), turned to -90 degrees
- moved U10 5.76 mm to (188.8, 31.1)
- moved C39 5.00 mm to (147.6, 88.9), turned to -90 degrees
- moved C11 1.98 mm to (93.2, 59.1)
Connections:
- J4 pad 2: Dout -> Net-(J4-Pad2)
- J4 pad 3: SCLK -> SDA
- J4 pad 4: RCLK -> SCL
- J4 pad 5: SER -> Net-(J4-Pad5)
- J5 pad 1: Net-(J5-Pad1) -> Net-(J4-Pad1)
- J5 pad 3: SCLK -> SDA
- J5 pad 4: RCLK -> SCL
- J5 pad 5: Dout -> Net-(J5-Pad5)
- U10 pad 1: Qb -> GND
- U10 pad 10: Vcc -> Qf
- U10 pad 11: SCLK -> Net-(U10-Pad11)
- U10 pad 12: RCLK -> Net-(U10-Pad12)
- U10 pad 13: GND -> Net-(U10-Pad13)
- U10 pad 14: SER -> SCL
- U10 pad 15: Qa -> SDA
- U10 pad 2: Qc -> GND
- U10 pad 3: Qd -> GND
- U10 pad 4: Qe -> Qa
- U10 pad 5: Qf -> Qb
- U10 pad 6: Qg -> Qc
- U10 pad 7: Qh -> Qd
- U10 pad 9: Net-(U10-Pad9) -> Qe
- U11 pad 1: Net-(U11-Pad1) -> Vcc
- U11 pad 10: Vcc -> Ql
- U11 pad 11: SCLK -> Qj
- U11 pad 12: RCLK -> Qi
- U11 pad 13: GND -> Net-(U11-Pad13)
- U11 pad 14: Net-(U10-Pad9) -> SCL
- U11 pad 15: Net-(U11-Pad15) -> SDA
- U11 pad 2: Net-(U11-Pad2) -> GND
- U11 pad 3: Net-(U11-Pad3) -> GND
- U11 pad 4: Qk -> Qg
- U11 pad 5: Ql -> Qh
- U11 pad 6: Qj -> Qm
- U11 pad 7: Qi -> Qn
- U11 pad 9: Dout -> Qk
Routing:
- net SDA: track 0.00 -> 88.8 mm, vias 0 -> 2
- net Qm: track 0.00 -> 73.6 mm, vias 0 -> 2
- net SCL: track 0.00 -> 62.9 mm, vias 0 -> 1
- net Qn: track 0.00 -> 61.1 mm, vias 0 -> 2
- net Dout: track 55.3 -> 0.00 mm
- net Net-(C49-Pad1): track 98.1 -> 150.4 mm
- net Qh: track 183.1 -> 134.7 mm, vias 2 -> 4
- net Net-(C62-Pad1): track 74.7 -> 120.5 mm
- net SCLK: track 44.7 -> 0.00 mm
- net Qg: track 187.5 -> 143.3 mm, vias 2 -> 5
- net RCLK: track 41.6 -> 0.00 mm
- net Qf: track 161.5 -> 178.3 mm
- net Net-(U10-Pad9): track 12.2 -> 0.00 mm
- net Vcc: track 65.8 -> 77.3 mm
- net Net-(C35-Pad1): track 31.0 -> 19.7 mm
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Other:
- net class Default removed
- net class smd removed
- net class smd2 removed
- net class smd3 removed
- rule pad_to_mask_clearance: 0.051 -> 0
